Commit message: add new spirit urdf

File: spirit_rl/resources/spirit40_old.urdf (robot description, URDF)
Before this commit: robot ngr, 17 links, 16 joints
Joints:
- joint 0: limit lower=-6.28318530718 upper=6.28318530718 effort=21 velocity=37.7 -> lower=-6.28318530718 upper=6.28318530718 effort=40 velocity=30
- joint 1: limit lower=0 upper=3.14159265359 effort=32 velocity=25.67 -> lower=0 upper=3.14159265359 effort=40 velocity=30
- joint 10: limit lower=-0.707 upper=0.707 effort=21 velocity=37.7 -> lower=-0.707 upper=0.707 effort=40 velocity=30
- joint 11: limit lower=-0.707 upper=0.707 effort=21 velocity=37.7 -> lower=-0.707 upper=0.707 effort=40 velocity=30
- joint 2: limit lower=-6.28318530718 upper=6.28318530718 effort=21 velocity=37.7 -> lower=-6.28318530718 upper=6.28318530718 effort=40 velocity=30
- joint 3: limit lower=0 upper=3.14159265359 effort=32 velocity=25.67 -> lower=0 upper=3.14159265359 effort=40 velocity=30
- joint 4: limit lower=-6.28318530718 upper=6.28318530718 effort=21 velocity=37.7 -> lower=-6.28318530718 upper=6.28318530718 effort=40 velocity=30
- joint 5: limit lower=0 upper=3.14159265359 effort=32 velocity=25.67 -> lower=0 upper=3.14159265359 effort=40 velocity=30
- joint 6: limit lower=-6.28318530718 upper=6.28318530718 effort=21 velocity=37.7 -> lower=-6.28318530718 upper=6.28318530718 effort=40 velocity=30
- joint 7: limit lower=0 upper=3.14159265359 effort=32 velocity=25.67 -> lower=0 upper=3.14159265359 effort=40 velocity=30
- joint 8: limit lower=-0.707 upper=0.707 effort=21 velocity=37.7 -> lower=-0.707 upper=0.707 effort=40 velocity=30
- joint 9: limit lower=-0.707 upper=0.707 effort=21 velocity=37.7 -> lower=-0.707 upper=0.707 effort=40 velocity=30
